File: Advanced Flash/SNES_AdvancedFlash_1-2.kicad_sch (KiCad schematic)
At the start: 34 parts, among them J1 Conn_02x03_Odd_Even, P1 SNES_Cartridge, SW1 SW_SPST, SW3 SW_SPST, SW4 SW_DIP_x02, SW5 SW_DIP_x02, U14 74HC74, U15 74AHC1G126, U1A1 PIC12F629, U1B1 PIC12F629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

Commit message: Add files via upload
Other:
- company: https://github.com/MouseBiteLabs -> https://github.com/MouseBiteLabs/Super-Nintendo-Cartridges
Changed lines of the file:
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@@
 	(title_block
 		(title "SNES Advanced Flash Cartridge")
-		(date "2024-08-09")
-		(rev "1.1")
-		(company "https://github.com/MouseBiteLabs")
+		(date "2024-09-18")
+		(rev "1.2")
+		(company "https://github.com/MouseBiteLabs/Super-Nintendo-Cartridges")
 	)
 	(bus_alias "COMMON_BUS"
