File: Advanced UV/RAM.kicad_sch (KiCad schematic)
At the start: 30 parts, among them Q1A 2N3904, Q1B MMBT3904, Q2 2N3904, U5 AS6C1008

Commit message: Add files via upload
Parts:
- renumbered CB1 to CB
Changed lines of the file:
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@@
 		(on_board yes)
 		(dnp no)
-		(property "Reference" "CB1"
+		(property "Reference" "CB"
 			(at 240.538 149.86 0)
 			(effects
@@
 			(project "SNES_Advanced_UV_1-0"
 				(path "/174e013e-6c2d-4e07-a41c-d66da3153f42/e5c4dfa1-4c7d-41d9-89a0-07b7dfe0aa1c"
-					(reference "CB1")
+					(reference "CB")
 					(unit 1)
 				)
