File: Advanced UV/SNES_Advanced_UV_1-0_new.kicad_pcb (KiCad board)
At the start: 2 copper layers, 116.2 x 68.2 mm, 65 parts, among them P1 SNES_Cartridge, Q1A 2N3904, Q1B MMBT3904, Q2 2N3904, U10 74HC74, U2A PIC12F629, U2B PIC12F629, U3H 27C322, U3L 27C322, U4H 27C322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

Commit message: Add files via upload
Parts:
- added G***: LOGO, LOGO, F.Cu at (195.8, 126.2)
