File: Advanced UV/SNES_Advanced_UV_1-0_new.kicad_sch (KiCad schematic)
At the start: 21 parts, among them P1 SNES_Cartridge, U10 74HC74, U2A PIC12F629, U2B PIC12F629, U6 74CBTLV3257, U7 74CBTLV3257, U8H 74LS139, U8L 74LS139, U9 74LS139

Commit message: Add files via upload
Connections:
- net CIC.D_{0}: now also P1.24 (CIC_{D1}), U2A.6 (GP1), U2B.6 (GP1); no longer P1.55 (CIC_{D0}), U2A.7 (GP0), U2B.7 (GP0)
- net CIC.D_{1}: now also P1.55 (CIC_{D0}), U2A.7 (GP0), U2B.7 (GP0); no longer P1.24 (CIC_{D1}), U2A.6 (GP1), U2B.6 (GP1)
Changed lines of the file:
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@@
 		)
 	)
-	(label "CIC.D_{0}"
+	(label "CIC.D_{1}"
 		(at 25.4 121.92 0)
 		(fields_autoplaced yes)
@@
 		)
 	)
-	(label "CIC.D_{1}"
+	(label "CIC.D_{0}"
 		(at 29.21 85.09 0)
 		(fields_autoplaced yes)
@@
 		)
 	)
-	(label "CIC.D_{0}"
+	(label "CIC.D_{1}"
 		(at 71.12 85.09 180)
 		(fields_autoplaced yes)
@@
 		)
 	)
-	(label "CIC.D_{1}"
+	(label "CIC.D_{0}"
 		(at 25.4 124.46 0)
 		(fields_autoplaced yes)
