File: Basic UV/SNES_Basic_UV_1-1.kicad_pcb (KiCad board)
At the start: 2 copper layers, 110.2 x 66.8 mm, 62 parts, among them P1 SNES_Cartridge, Q1A1 2N3904, Q1B1 MMBT3904, Q2 2N3904, U2A1 PIC12F629, U2B1 PIC12F629, U2C1 CIC, U3H1 SNES Mask ROM, U3L1 SNES Mask ROM, U4H1 27C160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

Commit message: Add files via upload
Parts:
- added SJ19: Jumper_3_Open, Bucketmouse:SJ_2, B.Cu at (145.8, 99.6)
Connections:
- TP2 pad 1: /~{WR} -> Net-(SJ19-A)
- TP3 pad 1: /~{WR} -> Net-(SJ19-B)
Routing:
- net Net-(SJ19-A): track 0.00 -> 10.7 mm
- net Net-(SJ19-B): track 0.00 -> 7.30 mm
- net /~{WR}: track 122.5 -> 129.2 mm, vias 4 -> 6
- net /BA_{6}: track 188.8 -> 185.9 mm
- net /D_{3}: track 77.4 -> 77.9 mm, vias 0 -> 2
- net GND: vias 104 -> 114
