File: Basic UV/RAM.kicad_sch (KiCad schematic)
At the start: 23 parts, among them Q1A1 2N3904, Q1B1 MMBT3904, Q2 2N3904, U5 AS6C1008

Commit message: Add files via upload
Parts:
- renumbered CB1 to CB, Q1A1 to Q1A, Q1B1 to Q1B
Changed lines of the file:
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@@
 (kicad_sch
-	(version 20231120)
+	(version 20250114)
 	(generator "eeschema")
-	(generator_version "8.0")
+	(generator_version "9.0")
 	(paper "A4")
 	(title_block
@@
 		(comment 2 "v1.1: Swap OEM CIC D0 and D1 pins, fix MAD-1 wiring, add selection for 27C160 modes")
 	)
+	(text "LOROM\n\n\n\n\nHIROM"
+		(exclude_from_sim no)
+		(at 112.268 136.144 0)
+		(effects
+			(font
+				(size 1.27 1.27)
+			)
+			(justify right)
+		)
+	)
+	(text "LOROM\n\n\n\n\nHIROM"
+		(exclude_from_sim no)
+		(at 76.708 156.464 0)
+		(effects
+			(font
+				(size 1.27 1.27)
+			)
+			(justify right)
+		)
+	)
+	(text "LOROM\n\n\n\n\nHIROM"
+		(exclude_from_sim no)
+		(at 58.928 169.164 0)
+		(effects
+			(font
+				(size 1.27 1.27)
+			)
+			(justify right)
+		)
+	)
+	(text "LOROM\n\n\n\n\nHIROM"
+		(exclude_from_sim no)
+		(at 94.488 146.304 0)
+		(effects
+			(font
+				(size 1.27 1.27)
+			)
+			(justify right)
+		)
+	)
 	(junction
 		(at 215.9 38.1)
@@
 		)
 	)
-	(text "LOROM\n\n\n\n\nHIROM"
-		(exclude_from_sim no)
-		(at 112.268 136.144 0)
-		(effects
-			(font
-				(size 1.27 1.27)
-			)
-			(justify right)
-		)
-	)
-	(text "LOROM\n\n\n\n\nHIROM"
-		(exclude_from_sim no)
-		(at 76.708 156.464 0)
-		(effects
-			(font
-				(size 1.27 1.27)
-			)
-			(justify right)
-		)
-	)
-	(text "LOROM\n\n\n\n\nHIROM"
-		(exclude_from_sim no)
-		(at 58.928 169.164 0)
-		(effects
-			(font
-				(size 1.27 1.27)
-			)
-			(justify right)
-		)
-	)
-	(text "LOROM\n\n\n\n\nHIROM"
-		(exclude_from_sim no)
-		(at 94.488 146.304 0)
-		(effects
-			(font
-				(size 1.27 1.27)
-			)
-			(justify right)
-		)
-	)
 	(label "~{CE}_{SRAM}"
 		(at 234.95 118.11 180)
-		(fields_autoplaced yes)
 		(effects
 			(font
@@
 	(label "A_{3}"
 		(at 40.64 102.87 0)
-		(fields_autoplaced yes)
 		(effects
 			(font
@@
 	(label "D_{4}"
 		(at 234.95 105.41 180)
-		(fields_autoplaced yes)
 		(effects
 			(font
@@
 	(label "D_{6}"
 		(at 234.95 110.49 180)
-		(fields_autoplaced yes)
 		(effects
 			(font
@@
 	(label "D_{7}"
 		(at 234.95 113.03 180)
-		(fields_autoplaced yes)
 		(effects
 			(font
@@
 	(label "A_{4}"
 		(at 40.64 105.41 0)
-		(fields_autoplaced yes)
 		(effects
 			(font
@@
 	(label "A_{12}"
 		(at 40.64 125.73 0)
-		(fields_autoplaced yes)
 		(effects
 			(font
@@
 	(label "A_{2}"
 		(at 40.64 100.33 0)
-		(fields_autoplaced yes)
 		(effects
 			(font
@@
 	(label "~{RESET}"
 		(at 176.53 44.45 0)
-		(fields_autoplaced yes)
 		(effects
 			(font
@@
 	(label "A_{11}"
 		(at 40.64 123.19 0)
-		(fields_autoplaced yes)
 		(effects
 			(font
@@
 	(label "A_{1}"
 		(at 40.64 97.79 0)
-		(fields_autoplaced yes)
 		(effects
 			(font
@@
 	(label "~{CE}_{SRAM}"
 		(at 240.03 38.1 180)
-		(fields_autoplaced yes)
 		(effects
 			(font
@@
 	(label "~{RESET}"
 		(at 109.22 44.45 0)
-		(fields_autoplaced yes)
 		(effects
 			(font
@@
 	(label "A_{0}"
 		(at 40.64 95.25 0)
-		(fields_autoplaced yes)
 		(effects
 			(font
@@
 	(label "A_{9}"
 		(at 40.64 118.11 0)
-		(fields_autoplaced yes)
 		(effects
 			(font
@@
 	(label "RA_{14}"
 		(at 187.96 130.81 0)
-		(fields_autoplaced yes)
 		(effects
 			(font
@@
 	(label "RA_{12}"
 		(at 187.96 125.73 0)
-		(fields_autoplaced yes)
 		(effects
 			(font
@@
 	(label "A_{7}"
 		(at 40.64 113.03 0)
-		(fields_autoplaced yes)
 		(effects
 			(font
@@
 	(label "D_{3}"
 		(at 234.95 102.87 180)
-		(fields_autoplaced yes)
 		(effects
 			(font
@@
 	(label "RA_{11}"
 		(at 187.96 123.19 0)
-		(fields_autoplaced yes)
 		(effects
 			(font
@@
 	(label "RA_{15}"
 		(at 187.96 133.35 0)
-		(fields_autoplaced yes)
 		(effects
 			(font
@@
 	(label "~{RD}"
 		(at 234.95 125.73 180)
-		(fields_autoplaced yes)
 		(effects
 			(font
@@
 	(label "D_{5}"
 		(at 234.95 107.95 180)
-		(fields_autoplaced yes)
 		(effects
 			(font
@@
 	(label "BA_{3}"
 		(at 40.64 140.97 0)
-		(fields_autoplaced yes)
 		(effects
 			(font
@@
 	(label "BA_{0}"
 		(at 40.64 133.35 0)
-		(fields_autoplaced yes)
 		(effects
 			(font
@@
 	(label "RA_{13}"
 		(at 187.96 128.27 0)
-		(fields_autoplaced yes)
 		(effects
 			(font
@@
 	(label "BA_{1}"
 		(at 40.64 135.89 0)
-		(fields_autoplaced yes)
 		(effects
 			(font
@@
 	(label "BA_{2}"
 		(at 40.64 138.43 0)
-		(fields_autoplaced yes)
 		(effects
 			(font
@@
 	(label "A_{14}"
 		(at 40.64 130.81 0)
-		(fields_autoplaced yes)
 		(effects
 			(font
@@
 	(label "A_{5}"
 		(at 40.64 107.95 0)
-		(fields_autoplaced yes)
 		(effects
 			(font
@@
 	(label "A_{8}"
 		(at 40.64 115.57 0)
-		(fields_autoplaced yes)
 		(effects
 			(font
@@
 	(label "~{WR}"
 		(at 234.95 128.27 180)
-		(fields_autoplaced yes)
 		(effects
 			(font
@@
 	(label "D_{2}"
 		(at 234.95 100.33 180)
-		(fields_autoplaced yes)
 		(effects
 			(font
@@
 	(label "D_{0}"
 		(at 234.95 95.25 180)
-		(fields_autoplaced yes)
 		(effects
 			(font
@@
 	(label "A_{6}"
 		(at 40.64 110.49 0)
-		(fields_autoplaced yes)
 		(effects
 			(font
@@
 	(label "A_{13}"
 		(at 40.64 128.27 0)
-		(fields_autoplaced yes)
 		(effects
 			(font
@@
 	(label "D_{1}"
 		(at 234.95 97.79 180)
-		(fields_autoplaced yes)
 		(effects
 			(font
@@
 	(label "A_{10}"
 		(at 40.64 120.65 0)
-		(fields_autoplaced yes)
 		(effects
 			(font
@@
 	(label "RA_{16}"
 		(at 187.96 135.89 0)
-		(fields_autoplaced yes)
 		(effects
 			(font
@@
 		(shape input)
 		(at 187.96 66.04 180)
-		(fields_autoplaced yes)
 		(effects
 			(font
@@
 		(shape input)
 		(at 187.96 62.23 180)
-		(fields_autoplaced yes)
 		(effects
 			(font
@@
 		(shape bidirectional)
 		(at 35.56 71.12 180)
-		(fields_autoplaced yes)
 		(effects
 			(font
@@
 		(on_board yes)
 		(dnp no)
-		(property "Reference" "Q1B1"
+		(property "Reference" "Q1B"
 			(at 216.408 50.8 0)
 			(effects
@@
 			(project ""
 				(path "/174e013e-6c2d-4e07-a41c-d66da3153f42/e5c4dfa1-4c7d-41d9-89a0-07b7dfe0aa1c"
-					(reference "Q1B1")
+					(reference "Q1B")
 					(unit 1)
 				)
@@
 		(on_board yes)
 		(dnp no)
-		(property "Reference" "CB1"
+		(property "Reference" "CB"
 			(at 240.538 149.86 0)
 			(effects
@@
 			(project "SNES_Advanced_UV_1-0"
 				(path "/174e013e-6c2d-4e07-a41c-d66da3153f42/e5c4dfa1-4c7d-41d9-89a0-07b7dfe0aa1c"
-					(reference "CB1")
+					(reference "CB")
 					(unit 1)
 				)
@@
 		(on_board yes)
 		(dnp no)
-		(property "Reference" "Q1A1"
+		(property "Reference" "Q1A"
 			(at 225.552 40.64 0)
 			(effects
@@
 			(project ""
 				(path "/174e013e-6c2d-4e07-a41c-d66da3153f42/e5c4dfa1-4c7d-41d9-89a0-07b7dfe0aa1c"
-					(reference "Q1A1")
+					(reference "Q1A")
 					(unit 1)
 				)
