File: Basic UV/ROM.kicad_sch (KiCad schematic)
At the start: 14 parts, among them U3H1 SNES Mask ROM, U3L1 SNES Mask ROM, U4H1 27C160, U4L1 27C160

Commit message: Add files via upload
Parts:
- added SJ19: Jumper_3_Open, Bucketmouse:SJ_2, symbol Jumper:Jumper_3_Open
Connections:
- net ~{WR}: now also SJ19.2 (C); no longer TP2.1, TP3.1
- new net: SJ19.3 (B), TP3.1
- new net: SJ19.1 (A), TP2.1
Other:
- note added: "LOROM HIROM"
- moved on the sheet: TP1, TP2, TP3
Changed lines of the file:
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@@
 	(title_block
 		(title "SNES Basic UV Cartridge")
-		(date "2025-11-15")
+		(date "2025-11-17")
 		(rev "v1.0")
 		(company "https://github.com/MouseBiteLabs/Super-Nintendo-Cartridges")
@@
 	)
 	(junction
-		(at 35.56 44.45)
-		(diameter 0)
-		(color 0 0 0 0)
-	)
-	(junction
 		(at 58.42 158.75)
 		(diameter 0)
@@
 	)
 	(junction
-		(at 40.64 44.45)
+		(at 36.83 44.45)
 		(diameter 0)
 		(color 0 0 0 0)
@@
 	(wire
 		(pts
-			(xy 30.48 44.45) (xy 35.56 44.45)
+			(xy 220.98 82.55) (xy 237.49 82.55)
 		)
 		(stroke
@@
 	(wire
 		(pts
-			(xy 220.98 82.55) (xy 237.49 82.55)
+			(xy 105.41 132.08) (xy 58.42 132.08)
 		)
 		(stroke
@@
 	(wire
 		(pts
-			(xy 105.41 132.08) (xy 58.42 132.08)
+			(xy 29.21 44.45) (xy 36.83 44.45)
 		)
 		(stroke
@@
 	(wire
 		(pts
+			(xy 36.83 44.45) (xy 36.83 48.26)
+		)
+		(stroke
+			(width 0)
+			(type default)
+		)
+	)
+	(wire
+		(pts
 			(xy 109.22 93.98) (xy 109.22 132.08)
 		)
@@
 	(wire
 		(pts
+			(xy 29.21 52.07) (xy 30.48 52.07)
+		)
+		(stroke
+			(width 0)
+			(type default)
+		)
+	)
+	(wire
+		(pts
 			(xy 157.48 105.41) (xy 173.99 105.41)
 		)
@@
 	(wire
 		(pts
+			(xy 36.83 44.45) (xy 45.72 44.45)
+		)
+		(stroke
+			(width 0)
+			(type default)
+		)
+	)
+	(wire
+		(pts
 			(xy 247.65 113.03) (xy 247.65 114.3)
 		)
@@
 	(wire
 		(pts
-			(xy 35.56 44.45) (xy 40.64 44.45)
-		)
-		(stroke
-			(width 0)
-			(type default)
-		)
-	)
-	(wire
-		(pts
 			(xy 101.6 78.74) (xy 113.03 78.74)
 		)
@@
 	(wire
 		(pts
+			(xy 43.18 52.07) (xy 44.45 52.07)
+		)
+		(stroke
+			(width 0)
+			(type default)
+		)
+	)
+	(wire
+		(pts
 			(xy 157.48 64.77) (xy 173.99 64.77)
 		)
@@
 	(wire
 		(pts
-			(xy 40.64 44.45) (xy 45.72 44.45)
-		)
-		(stroke
-			(width 0)
-			(type default)
-		)
-	)
-	(wire
-		(pts
 			(xy 220.98 49.53) (xy 237.49 49.53)
 		)
@@
 		)
 	)
+	(text "LOROM\n\n\n\n\nHIROM"
+		(exclude_from_sim no)
+		(at 36.83 52.578 90)
+		(effects
+			(font
+				(size 1.27 1.27)
+			)
+			(justify right)
+		)
+	)
 	(label "A_{11}"
 		(at 50.8 81.28 0)
@@
 	(symbol
 		(lib_id "Connector:TestPoint")
-		(at 40.64 44.45 0)
+		(at 44.45 52.07 0)
 		(mirror y)
 		(unit 1)
@@
 		(dnp no)
 		(property "Reference" "TP3"
-			(at 40.64 39.116 0)
+			(at 44.45 46.736 0)
 			(effects
 				(font
@@
 		)
 		(property "Value" "TPB1,27"
-			(at 40.64 39.37 0)
+			(at 44.45 46.99 0)
 			(effects
 				(font
@@
 		)
 		(property "Footprint" "Bucketmouse:TestPoint_THTPad_D1.5mm_Drill0.7mm"
-			(at 35.56 44.45 0)
+			(at 39.37 52.07 0)
 			(effects
 				(font
@@
 		)
 		(property "Datasheet" "~"
-			(at 35.56 44.45 0)
+			(at 39.37 52.07 0)
 			(effects
 				(font
@@
 		)
 		(property "Description" "test point"
-			(at 40.64 44.45 0)
+			(at 44.45 52.07 0)
 			(effects
 				(font
@@
 	)
 	(symbol
+		(lib_id "Jumper:Jumper_3_Open")
+		(at 36.83 52.07 0)
+		(mirror x)
+		(unit 1)
+		(exclude_from_sim yes)
+		(in_bom no)
+		(on_board yes)
+		(dnp no)
+		(property "Reference" "SJ19"
+			(at 36.83 53.848 90)
+			(effects
+				(font
+					(size 1.27 1.27)
+				)
+				(justify left)
+			)
+		)
+		(property "Value" "Jumper_3_Open"
+			(at 38.0999 54.61 90)
+			(effects
+				(font
+					(size 1.27 1.27)
+				)
+				(justify left)
+				(hide yes)
+			)
+		)
+		(property "Footprint" "Bucketmouse:SJ_2"
+			(at 36.83 52.07 0)
+			(effects
+				(font
+					(size 1.27 1.27)
+				)
+				(hide yes)
+			)
+		)
+		(property "Datasheet" "~"
+			(at 36.83 52.07 0)
+			(effects
+				(font
+					(size 1.27 1.27)
+				)
+				(hide yes)
+			)
+		)
+		(property "Description" "Jumper, 3-pole, both open"
+			(at 36.83 52.07 0)
+			(effects
+				(font
+					(size 1.27 1.27)
+				)
+				(hide yes)
+			)
+		)
+		(pin "1"
+		)
+		(pin "2"
+		)
+		(pin "3"
+		)
+		(instances
+			(project "SNES_Basic_UV_1-1"
+				(path "/174e013e-6c2d-4e07-a41c-d66da3153f42/3fcebb72-8a4d-4e82-b228-0c6cfb7b62ec"
+					(reference "SJ19")
+					(unit 1)
+				)
+			)
+		)
+	)
+	(symbol
 		(lib_id "power:GND")
 		(at 185.42 114.3 0)
@@
 	(symbol
 		(lib_id "Connector:TestPoint")
-		(at 30.48 44.45 0)
+		(at 29.21 44.45 0)
 		(mirror y)
 		(unit 1)
@@
 		(dnp no)
 		(property "Reference" "TP1"
-			(at 30.48 39.116 0)
+			(at 29.21 39.116 0)
 			(effects
 				(font
@@
 		)
 		(property "Value" "TPB1,27"
-			(at 30.48 39.37 0)
+			(at 29.21 39.37 0)
 			(effects
 				(font
@@
 		)
 		(property "Footprint" "Bucketmouse:TestPoint_THTPad_D1.5mm_Drill0.7mm"
-			(at 25.4 44.45 0)
+			(at 24.13 44.45 0)
 			(effects
 				(font
@@
 		)
 		(property "Datasheet" "~"
-			(at 25.4 44.45 0)
+			(at 24.13 44.45 0)
 			(effects
 				(font
@@
 		)
 		(property "Description" "test point"
-			(at 30.48 44.45 0)
+			(at 29.21 44.45 0)
 			(effects
 				(font
@@
 	(symbol
 		(lib_id "Connector:TestPoint")
-		(at 35.56 44.45 0)
+		(at 29.21 52.07 0)
 		(mirror y)
 		(unit 1)
@@
 		(dnp no)
 		(property "Reference" "TP2"
-			(at 35.56 39.116 0)
+			(at 29.21 46.736 0)
 			(effects
 				(font
@@
 		)
 		(property "Value" "TPB1,27"
-			(at 35.56 39.37 0)
+			(at 29.21 46.99 0)
 			(effects
 				(font
@@
 		)
 		(property "Footprint" "Bucketmouse:TestPoint_THTPad_D1.5mm_Drill0.7mm"
-			(at 30.48 44.45 0)
+			(at 24.13 52.07 0)
 			(effects
 				(font
@@
 		)
 		(property "Datasheet" "~"
-			(at 30.48 44.45 0)
+			(at 24.13 52.07 0)
 			(effects
 				(font
@@
 		)
 		(property "Description" "test point"
-			(at 35.56 44.45 0)
+			(at 29.21 52.07 0)
 			(effects
 				(font

Commit message: Add files via upload
Parts:
- renumbered U3H1 to U3H, U3L1 to U3L, U4H1 to U4H, U4L1 to U4L
