File: Basic UV/SNES_Basic_UV_1-1.kicad_sch (KiCad schematic)
At the start: 22 parts, among them P1 SNES_Cartridge, U2A1 PIC12F629, U2B1 PIC12F629, U2C1 CIC, U6H1 MAD-1, U6L1 MAD-1, U8H1 74LS139, U8L1 74LS139

Commit message: Add files via upload
Parts:
- renumbered C22 to C2
Changed lines of the file:
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@@
 	(title_block
 		(title "SNES Basic UV Cartridge")
-		(date "2025-11-15")
+		(date "2025-11-17")
 		(rev "v1.0")
 		(company "https://github.com/MouseBiteLabs/Super-Nintendo-Cartridges")
@@
 		(on_board yes)
 		(dnp no)
-		(property "Reference" "C22"
+		(property "Reference" "C2"
 			(at 67.31 126.9999 0)
 			(effects
@@
 			(project "SNES_Basic_UV_1-0"
 				(path "/174e013e-6c2d-4e07-a41c-d66da3153f42"
-					(reference "C22")
+					(reference "C2")
 					(unit 1)
 				)

Commit message: Add files via upload
Parts:
- renumbered U2A1 to U2A, U2B1 to U2B, U2C1 to U2C, U6H1 to U6H, U6L1 to U6L, U8H1 to U8H, U8L1 to U8L
